File: hardware/KiCad/PT2258.kicad_sch (KiCad schematic)
At the start: 53 parts, among them J1 Conn_01x03_Pin, J10 SpeakON_NL2, J11 SpeakON_NL2, J12 SpeakON_NL2, J13 Conn_01x02, J2 Conn_01x03_Pin, J3 Conn_01x03_Pin, J4 Conn_01x03_Pin, J5 SpeakON_NL2, J6 SpeakON_NL2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

Commit message: Add files via upload
Parts:
- added C16, C18, C20, C28, C29, C30, C31, C32: 10n, symbol Device:C
- added C26, C27: 10µF, Capacitor_THT:CP_Radial_D6.3mm_P2.50mm, symbol Device:C_Polarized
- added D1, D2: 1N4005, symbol Device:D
- added R15, R16: 2k2, symbol Device:R
- added R17, R18, R19, R20, R21, R22, R23, R24: 100k, symbol Device:R
- added U3: ESP32-S3-DevKitC, PCM_Espressif:ESP32-S3-DevKitC, symbol Espressif:ESP32-S3-DevKitC
- added U4: TFT_320x240, z_Devices:TFT-320x240, symbol tft_320x240:TFT_320x240
- renumbered R23 to R27, R24 to R28
Connections:
- net +20V: now also D1.1 (K)
- net +5V: now also C26.1, D1.2 (A), D2.1 (K), U3.21 (5V)
- net GNDA: now also C26.2, C27.2, U3.22 (GND), U3.23 (GND), U3.24 (GND), U3.44 (GND), U4.2 (GND)
- net T-RR: now reaches C6.2, J3.3 (Pin_3), R6.1
- net T-RR: now also C31.2
- net at U1.6 (SCL), U2.6 (SCL): now also R16.2, U3.5 (GPIO5/ADC1_CH4)
- net at U1.7 (SDA), U2.7 (SDA): now also R15.2, U3.6 (GPIO6/ADC1_CH5)
- net T-RL: now reaches C5.2, J3.1 (Pin_1), R5.1
- net T-RL: now also C20.2
- net T-FR: now reaches C2.2, J1.3 (Pin_3), R2.1
- net T-FR: now also C29.2
- net T-SR: now reaches C4.2, J2.3 (Pin_3), R4.1
- net T-SR: now also C30.2
- net T-C: now reaches C17.2, J4.1 (Pin_1), R13.1
- net T-C: now also C28.2
- net T-SUB: now reaches C15.2, J4.3 (Pin_3), R14.1
- net T-SUB: now also C32.2
- net T-FL: now reaches C1.2, J1.1 (Pin_1), R1.1
- net T-FL: now also C16.2
- net T-SL: now reaches C3.2, J2.1 (Pin_1), R3.1
- net T-SL: now also C18.2
- new net: R17.1, U3.27 (GPIO21)
- new net: C16.1, R17.2
- new net: R24.1, U3.28 (GPIO47)
- new net: C32.1, R24.2
- new net: R18.1, U3.32 (GPIO35)
- new net: C29.1, R18.2
- new net: R22.1, U3.30 (GPIO45)
- new net: C31.1, R22.2
- new net: C18.1, R19.2
- new net: U3.12 (GPIO8/ADC1_CH7), U4.5 (DC)
- new net: R23.1, U3.14 (GPIO46)
- new net: U3.15 (GPIO9/ADC1_CH8), U4.11
- new net: U3.16 (GPIO10/ADC1_CH9), U4.3 (CS)
- new net: U3.17 (GPIO11/ADC2_CH0), U4.4 (RST)
- new net: U3.18 (GPIO12/ADC2_CH1), U4.13, U4.9 (MISO)
- new net: U3.19 (GPIO13/ADC2_CH2), U4.12, U4.6 (MOSI)
- new net: U3.20 (GPIO14/ADC2_CH3), U4.10, U4.7 (SCK)
- new net: R19.1, U3.33 (GPIO36)
- new net: R20.1, U3.34 (GPIO37)
- new net: R21.1, U3.35 (GPIO38)
- new net: C28.1, R23.2
- new net: C20.1, R21.2
- new net: C30.1, R20.2
- new net +3.3V: C27.1, D2.2 (A), R15.1, R16.1, U3.1 (3V3), U3.2 (3V3), U4.1 (VCC), U4.8 (LED)
Other:
- note added: "100k"
- note added: "10n"
- note added: "Voltage regulator 3.3V"
- note added: "Voltage regulator 5V"
- moved on the sheet: C15, C17, J13, R13, R14
